File: Hardware/Breadboard Power Supply - SMD.sch (EAGLE design)
At the start: 25 parts, among them J1 POWER_JACKTYLERALT1, U1 V_REG_317SMD

Commit message: Fixed Review Issues
Added extra VCC and GND headers for stability. spaced out res along top
edge. removed weird tDocu lines. cleaned up repo
Parts:
- added JP6, JP7, JP8, JP9: M01PTH, SparkFun:M01PTH
Connections:
- net GND: now also JP6.1, JP9.1
- net VCC: now also JP7.1, JP8.1
Changed lines of the file:
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@@
 <grid distance="0.1" unitdist="inch" unit="inch" style="lines" multiple="1" display="no" altdistance="0.01" altunitdist="inch" altunit="inch"/>
 <layers>
-<layer number="1" name="Top" color="4" fill="1" visible="yes" active="no"/>
-<layer number="2" name="Route2" color="1" fill="3" visible="yes" active="no"/>
-<layer number="3" name="Route3" color="4" fill="3" visible="yes" active="no"/>
-<layer number="4" name="Route4" color="1" fill="4" visible="yes" active="no"/>
-<layer number="5" name="Route5" color="4" fill="4" visible="yes" active="no"/>
-<layer number="6" name="Route6" color="1" fill="8" visible="yes" active="no"/>
-<layer number="7" name="Route7" color="4" fill="8" visible="yes" active="no"/>
-<layer number="8" name="Route8" color="1" fill="2" visible="yes" active="no"/>
-<layer number="9" name="Route9" color="4" fill="2" visible="yes" active="no"/>
-<layer number="10" name="Route10" color="1" fill="7" visible="yes" active="no"/>
-<layer number="11" name="Route11" color="4" fill="7" visible="yes" active="no"/>
-<layer number="12" name="Route12" color="1" fill="5" visible="yes" active="no"/>
-<layer number="13" name="Route13" color="4" fill="5" visible="yes" active="no"/>
-<layer number="14" name="Route14" color="1" fill="6" visible="yes" active="no"/>
-<layer number="15" name="Route15" color="4" fill="6" visible="yes" active="no"/>
-<layer number="16" name="Bottom" color="1" fill="1" visible="yes" active="no"/>
-<layer number="17" name="Pads" color="2" fill="1" visible="yes" active="no"/>
-<layer number="18" name="Vias" color="2" fill="1" visible="yes" active="no"/>
-<layer number="19" name="Unrouted" color="6" fill="1" visible="yes" active="no"/>
-<layer number="20" name="Dimension" color="15" fill="1" visible="yes" active="no"/>
-<layer number="21" name="tPlace" color="16" fill="1" visible="yes" active="no"/>
-<layer number="22" name="bPlace" color="14" fill="1" visible="yes" active="no"/>
-<layer number="23" name="tOrigins" color="15" fill="1" visible="yes" active="no"/>
-<layer number="24" name="bOrigins" color="15" fill="1" visible="yes" active="no"/>
-<layer number="25" name="tNames" color="7" fill="1" visible="yes" active="no"/>
-<layer number="26" name="bNames" color="7" fill="1" visible="yes" active="no"/>
-<layer number="27" name="tValues" color="7" fill="1" visible="yes" active="no"/>
-<layer number="28" name="bValues" color="7" fill="1" visible="yes" active="no"/>
+<layer number="1" name="Top" color="4" fill="1" visible="no" active="no"/>
+<layer number="2" name="Route2" color="1" fill="3" visible="no" active="no"/>
+<layer number="3" name="Route3" color="4" fill="3" visible="no" active="no"/>
+<layer number="4" name="Route4" color="1" fill="4" visible="no" active="no"/>
+<layer number="5" name="Route5" color="4" fill="4" visible="no" active="no"/>
+<layer number="6" name="Route6" color="1" fill="8" visible="no" active="no"/>
+<layer number="7" name="Route7" color="4" fill="8" visible="no" active="no"/>
+<layer number="8" name="Route8" color="1" fill="2" visible="no" active="no"/>
+<layer number="9" name="Route9" color="4" fill="2" visible="no" active="no"/>
+<layer number="10" name="Route10" color="1" fill="7" visible="no" active="no"/>
+<layer number="11" name="Route11" color="4" fill="7" visible="no" active="no"/>
+<layer number="12" name="Route12" color="1" fill="5" visible="no" active="no"/>
+<layer number="13" name="Route13" color="4" fill="5" visible="no" active="no"/>
+<layer number="14" name="Route14" color="1" fill="6" visible="no" active="no"/>
+<layer number="15" name="Route15" color="4" fill="6" visible="no" active="no"/>
+<layer number="16" name="Bottom" color="1" fill="1" visible="no" active="no"/>
+<layer number="17" name="Pads" color="2" fill="1" visible="no" active="no"/>
+<layer number="18" name="Vias" color="2" fill="1" visible="no" active="no"/>
+<layer number="19" name="Unrouted" color="6" fill="1" visible="no" active="no"/>
+<layer number="20" name="Dimension" color="15" fill="1" visible="no" active="no"/>
+<layer number="21" name="tPlace" color="16" fill="1" visible="no" active="no"/>
+<layer number="22" name="bPlace" color="14" fill="1" visible="no" active="no"/>
+<layer number="23" name="tOrigins" color="15" fill="1" visible="no" active="no"/>
+<layer number="24" name="bOrigins" color="15" fill="1" visible="no" active="no"/>
+<layer number="25" name="tNames" color="7" fill="1" visible="no" active="no"/>
+<layer number="26" name="bNames" color="7" fill="1" visible="no" active="no"/>
+<layer number="27" name="tValues" color="7" fill="1" visible="no" active="no"/>
+<layer number="28" name="bValues" color="7" fill="1" visible="no" active="no"/>
 <layer number="29" name="tStop" color="7" fill="3" visible="no" active="no"/>
 <layer number="30" name="bStop" color="7" fill="6" visible="no" active="no"/>
@@
 <layer number="35" name="tGlue" color="7" fill="4" visible="no" active="no"/>
 <layer number="36" name="bGlue" color="7" fill="5" visible="no" active="no"/>
-<layer number="37" name="tTest" color="7" fill="1" visible="yes" active="no"/>
-<layer number="38" name="bTest" color="7" fill="1" visible="yes" active="no"/>
+<layer number="37" name="tTest" color="7" fill="1" visible="no" active="no"/>
+<layer number="38" name="bTest" color="7" fill="1" visible="no" active="no"/>
 <layer number="39" name="tKeepout" color="4" fill="11" visible="no" active="no"/>
 <layer number="40" name="bKeepout" color="1" fill="11" visible="no" active="no"/>
@@
 <layer number="44" name="Drills" color="7" fill="1" visible="no" active="no"/>
 <layer number="45" name="Holes" color="7" fill="1" visible="no" active="no"/>
-<layer number="46" name="Milling" color="3" fill="1" visible="yes" active="no"/>
-<layer number="47" name="Measures" color="7" fill="1" visible="yes" active="no"/>
-<layer number="48" name="Document" color="7" fill="1" visible="yes" active="no"/>
-<layer number="49" name="Reference" color="7" fill="1" visible="yes" active="no"/>
-<layer number="50" name="dxf" color="7" fill="1" visible="yes" active="no"/>
-<layer number="51" name="tDocu" color="6" fill="1" visible="yes" active="no"/>
-<layer number="52" name="bDocu" color="7" fill="1" visible="yes" active="no"/>
-<layer number="53" name="tGND_GNDA" color="7" fill="9" visible="yes" active="no"/>
-<layer number="54" name="bGND_GNDA" color="1" fill="9" visible="yes" active="no"/>
-<layer number="56" name="wert" color="7" fill="1" visible="yes" active="no"/>
+<layer number="46" name="Milling" color="3" fill="1" visible="no" active="no"/>
+<layer number="47" name="Measures" color="7" fill="1" visible="no" active="no"/>
+<layer number="48" name="Document" color="7" fill="1" visible="no" active="no"/>
+<layer number="49" name="Reference" color="7" fill="1" visible="no" active="no"/>
+<layer number="50" name="dxf" color="7" fill="1" visible="no" active="no"/>
+<layer number="51" name="tDocu" color="6" fill="1" visible="no" active="no"/>
+<layer number="52" name="bDocu" color="7" fill="1" visible="no" active="no"/>
+<layer number="53" name="tGND_GNDA" color="7" fill="9" visible="no" active="no"/>
+<layer number="54" name="bGND_GNDA" color="1" fill="9" visible="no" active="no"/>
+<layer number="56" name="wert" color="7" fill="1" visible="no" active="no"/>
 <layer number="91" name="Nets" color="2" fill="1" visible="yes" active="yes"/>
 <layer number="92" name="Busses" color="1" fill="1" visible="yes" active="yes"/>
@@
 <part name="U$4" library="SparkFun" deviceset="FIDUCIAL" device="1X2"/>
 <part name="LOGO1" library="SparkFun-Aesthetics" deviceset="OSHW-LOGO" device="S"/>
+<part name="JP6" library="SparkFun" deviceset="M01" device="PTH"/>
+<part name="JP7" library="SparkFun" deviceset="M01" device="PTH"/>
+<part name="JP8" library="SparkFun" deviceset="M01" device="PTH"/>
+<part name="JP9" library="SparkFun" deviceset="M01" device="PTH"/>
 </parts>
 <sheets>
@@
 <instance part="U$4" gate="G$1" x="243.84" y="27.94"/>
 <instance part="LOGO1" gate="G$1" x="124.46" y="12.7"/>
+<instance part="JP6" gate="G$1" x="170.18" y="55.88" rot="R180"/>
+<instance part="JP7" gate="G$1" x="170.18" y="66.04" rot="R180"/>
+<instance part="JP8" gate="G$1" x="193.04" y="66.04" rot="R180"/>
+<instance part="JP9" gate="G$1" x="193.04" y="55.88" rot="R180"/>
 </instances>
 <busses>
@@
 <label x="114.3" y="55.88" size="1.778" layer="95"/>
 <pinref part="JP1" gate="G$1" pin="1"/>
+</segment>
+<segment>
+<wire x1="185.42" y1="55.88" x2="180.34" y2="55.88" width="0.1524" layer="91"/>
+<label x="180.34" y="55.88" size="1.778" layer="95"/>
+<pinref part="JP9" gate="G$1" pin="1"/>
+</segment>
+<segment>
+<wire x1="162.56" y1="55.88" x2="157.48" y2="55.88" width="0.1524" layer="91"/>
+<label x="157.48" y="55.88" size="1.778" layer="95"/>
+<pinref part="JP6" gate="G$1" pin="1"/>
 </segment>
 </net>
@@
 <pinref part="JP2" gate="G$1" pin="1"/>
 </segment>
-</net>
+<segment>
+<wire x1="185.42" y1="66.04" x2="180.34" y2="66.04" width="0.1524" layer="91"/>
+<label x="180.34" y="66.04" size="1.778" layer="95"/>
+<pinref part="JP8" gate="G$1" pin="1"/>
+</segment>
+<segment>
+<wire x1="162.56" y1="66.04" x2="157.48" y2="66.04" width="0.1524" layer="91"/>
+<label x="157.48" y="66.04" size="1.778" layer="95"/>
+<pinref part="JP7" gate="G$1" pin="1"/>
+</segment>
+</net>

Commit message: Updated Footprints
Updated footprints on the Diode/PTC/BarrelJack
Parts:
- F1: value PTCWIDE -> PTCSMD-W; device Testing:PTCWIDE -> SparkFun-PowerIC:PTCSMD-W
- J1: value POWER_JACKTYLERALT1 -> POWER_JACKSMD; device Testing:POWER_JACKTYLERALT1 -> SparkFun-Connectors:POWER_JACKSMD
Other:
- note added: "Revised by: Patrick Alberts"
- note removed: "(the previous FP was too tight and didn't allow part to sit flush on PCB)"
- note removed: "-changed to 0603 FPs"
- note removed: "-moved barrel jack up to avoid overhang"
- note removed: "-updated FP on barrel jack to use larger drill holes"
- note removed: "Changes to v13 (5/23/11):"
- note removed: "Revised by: T Talmage"
- moved on the sheet: JP6, JP7, JP8, JP9
Changed lines of the file:
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@@
 <part name="C3" library="SparkFun" deviceset="CAP" device="0603-CAP" value="0.1uF"/>
 <part name="U1" library="SparkFun" deviceset="V_REG_317" device="SMD"/>
-<part name="F1" library="Testing" deviceset="PTC" device="WIDE"/>
+<part name="F1" library="SparkFun-PowerIC" deviceset="PTC" device="SMD-W"/>
 <part name="RAW" library="SparkFun" deviceset="VCC" device="" value="RAW"/>
 <part name="P+3" library="SparkFun" deviceset="VCC" device=""/>
@@
 <part name="JP4" library="SparkFun" deviceset="M01" device="PTH"/>
 <part name="U$1" library="SparkFun" deviceset="LOGO-SFE" device="SK"/>
-<part name="J1" library="Testing" deviceset="POWER_JACK" device="TYLERALT1"/>
+<part name="J1" library="SparkFun-Connectors" deviceset="POWER_JACK" device="SMD"/>
 <part name="JP5" library="SparkFun" deviceset="M02" device="PTH"/>
 <part name="D1" library="Testing" deviceset="DIODE" device="SMA-TYLERALT1" value="1N4001"/>
@@
 <text x="147.32" y="83.82" size="1.778" layer="96">Open: 5V</text>
 <text x="167.64" y="10.16" size="1.778" layer="94">N. Seidle</text>
-<text x="251.46" y="182.88" size="1.778" layer="94">Changes to v13 (5/23/11):</text>
-<text x="251.46" y="180.34" size="1.778" layer="94">-updated FP on barrel jack to use larger drill holes</text>
-<text x="254" y="177.8" size="1.778" layer="94">(the previous FP was too tight and didn't allow part to sit flush on PCB)</text>
-<text x="251.46" y="172.72" size="1.778" layer="94">-changed to 0603 FPs</text>
-<text x="251.46" y="175.26" size="1.778" layer="94">-moved barrel jack up to avoid overhang</text>
-<text x="182.88" y="10.16" size="1.778" layer="94">Revised by: T Talmage</text>
+<text x="182.88" y="10.16" size="1.778" layer="94">Revised by: Patrick Alberts</text>
 </plain>
 <instances>
@@
 <instance part="U$4" gate="G$1" x="243.84" y="27.94"/>
 <instance part="LOGO1" gate="G$1" x="124.46" y="12.7"/>
-<instance part="JP6" gate="G$1" x="170.18" y="55.88" rot="R180"/>
-<instance part="JP7" gate="G$1" x="170.18" y="66.04" rot="R180"/>
-<instance part="JP8" gate="G$1" x="193.04" y="66.04" rot="R180"/>
-<instance part="JP9" gate="G$1" x="193.04" y="55.88" rot="R180"/>
+<instance part="JP6" gate="G$1" x="172.72" y="55.88" rot="R180"/>
+<instance part="JP7" gate="G$1" x="172.72" y="66.04" rot="R180"/>
+<instance part="JP8" gate="G$1" x="195.58" y="66.04" rot="R180"/>
+<instance part="JP9" gate="G$1" x="195.58" y="55.88" rot="R180"/>
 </instances>
 <busses>
@@
 </segment>
 <segment>
-<wire x1="142.24" y1="55.88" x2="137.16" y2="55.88" width="0.1524" layer="91"/>
-<label x="137.16" y="55.88" size="1.778" layer="95"/>
+<wire x1="142.24" y1="55.88" x2="139.7" y2="55.88" width="0.1524" layer="91"/>
 <pinref part="JP4" gate="G$1" pin="1"/>
+<label x="139.7" y="55.88" size="1.778" layer="95" rot="R180" xref="yes"/>
 </segment>
 <segment>
@@
 </segment>
 <segment>
-<wire x1="119.38" y1="55.88" x2="114.3" y2="55.88" width="0.1524" layer="91"/>
-<label x="114.3" y="55.88" size="1.778" layer="95"/>
+<wire x1="119.38" y1="55.88" x2="116.84" y2="55.88" width="0.1524" layer="91"/>
 <pinref part="JP1" gate="G$1" pin="1"/>
-</segment>
-<segment>
-<wire x1="185.42" y1="55.88" x2="180.34" y2="55.88" width="0.1524" layer="91"/>
-<label x="180.34" y="55.88" size="1.778" layer="95"/>
+<label x="116.84" y="55.88" size="1.778" layer="95" rot="R180" xref="yes"/>
+</segment>
+<segment>
+<wire x1="187.96" y1="55.88" x2="185.42" y2="55.88" width="0.1524" layer="91"/>
 <pinref part="JP9" gate="G$1" pin="1"/>
-</segment>
-<segment>
-<wire x1="162.56" y1="55.88" x2="157.48" y2="55.88" width="0.1524" layer="91"/>
-<label x="157.48" y="55.88" size="1.778" layer="95"/>
+<label x="185.42" y="55.88" size="1.778" layer="95" rot="R180" xref="yes"/>
+</segment>
+<segment>
+<wire x1="165.1" y1="55.88" x2="162.56" y2="55.88" width="0.1524" layer="91"/>
 <pinref part="JP6" gate="G$1" pin="1"/>
+<label x="162.56" y="55.88" size="1.778" layer="95" rot="R180" xref="yes"/>
 </segment>
 </net>
@@
 </segment>
 <segment>
-<wire x1="142.24" y1="66.04" x2="137.16" y2="66.04" width="0.1524" layer="91"/>
-<label x="137.16" y="66.04" size="1.778" layer="95"/>
+<wire x1="142.24" y1="66.04" x2="139.7" y2="66.04" width="0.1524" layer="91"/>
 <pinref part="JP3" gate="G$1" pin="1"/>
-</segment>
-<segment>
-<wire x1="119.38" y1="66.04" x2="114.3" y2="66.04" width="0.1524" layer="91"/>
-<label x="114.3" y="66.04" size="1.778" layer="95"/>
+<label x="139.7" y="66.04" size="1.778" layer="95" rot="R180" xref="yes"/>
+</segment>
+<segment>
+<wire x1="119.38" y1="66.04" x2="116.84" y2="66.04" width="0.1524" layer="91"/>
 <pinref part="JP2" gate="G$1" pin="1"/>
-</segment>
-<segment>
-<wire x1="185.42" y1="66.04" x2="180.34" y2="66.04" width="0.1524" layer="91"/>
-<label x="180.34" y="66.04" size="1.778" layer="95"/>
+<label x="116.84" y="66.04" size="1.778" layer="95" rot="R180" xref="yes"/>
+</segment>
+<segment>
+<wire x1="187.96" y1="66.04" x2="185.42" y2="66.04" width="0.1524" layer="91"/>
 <pinref part="JP8" gate="G$1" pin="1"/>
-</segment>
-<segment>
-<wire x1="162.56" y1="66.04" x2="157.48" y2="66.04" width="0.1524" layer="91"/>
-<label x="157.48" y="66.04" size="1.778" layer="95"/>
+<label x="185.42" y="66.04" size="1.778" layer="95" rot="R180" xref="yes"/>
+</segment>
+<segment>
+<wire x1="165.1" y1="66.04" x2="162.56" y2="66.04" width="0.1524" layer="91"/>
 <pinref part="JP7" gate="G$1" pin="1"/>
-</segment>
-</net>
+<label x="162.56" y="66.04" size="1.778" layer="95" rot="R180" xref="yes"/>
+</segment>
+</net>
